File: can.sch (EAGLE design)
At the start: 17 parts, among them IC2 MEGA8-P, Q1 16Mhz, Q2 10Mhz

Commit message: fix
Parts:
- added AN0, AN1, AN2, AN3: (no value), pinhead:PINHD-1X3
- added C5, C6, C7: .1nf, rcl:C-EU025-025X050
- added CF: 1nf, rcl:C-EU025-025X050
- added C_BYP: 0.1nf, rcl:C-EU025-025X050
- added IC1: 7805TV, linear:7805TV
- added ICSP: (no value), pinhead:PINHD-2X3
- added K2: G5LE, relay:G5LE
- added R5, R6: 10k, rcl:R-EU_0207/10
- added RA: (no value), con-ptr500:AK500/3
- added T1: (no value), transistor:BC548-NPN-TO92-CBE
- added TERM1: (no value), pinhead:PINHD-1X2
- added U1: ACS712ELCTR-05B-T, Allegro_By_element14_Batch_1:ACS712ELCTR-05B-T
- added X2: (no value), con-ptr500:AK500/2
- Q2: value 10Mhz -> 16Mhz
Connections:
- new net B0: AN0.2, IC2.PC0(ADC0)
- new net B1: AN1.2, IC2.PC1(ADC1)
- new net B2: AN2.2, IC2.PC2(ADC2)
- new net B3: AN3.2, IC2.PC3(ADC3)
- new net N$10: K21.2, T1.C
- new net N$16: R5.1, T1.B
- new net N$18: RA-2.KL, U1.IP+, U1.IP+_2
- new net N$19: K22.O, RA-1.KL
- new net N$20: K22.S, RA-3.KL
- new net N$21: IC2.PC6(/RESET), ICSP.5, R6.1
- new net N$22: IC2.PD0(RXD), TERM1.1
- new net N$23: IC2.PD1(TXD), TERM1.2
- new net N$24: IC2.PD6(AIN0), R5.2
- new net N$25: IC2.PD7(AIN1), U1.VIOUT
- new net N$26: CF.1, U1.FILTER
- new net N$27: K22.P, U1.IP-, U1.IP-_2
- new net N$29: C7.1, IC1.VI, X2-1.KL
- net GND: now also AN0.3, AN1.3, AN2.3, AN3.3, C5.1, C6.2, C7.2, CF.2, C_BYP.2, IC1.GND, T1.E, U1.GND, X2-2.KL
- net N$3: now also ICSP.4
- net N$6: now also ICSP.3
- net N$7: now also ICSP.2
- net VCC: now also AN0.1, AN1.1, AN2.1, AN3.1, C5.2, C6.1, C_BYP.1, IC1.VO, ICSP.1, K21.1, R6.2, U1.VCC
Other:
- moved on the sheet: R4

Commit message: fix
Parts:
- removed R4: 10k, rcl:R-EU_0207/10
- removed X1: (no value), con-ptr500:AK500/2
- added CF1: 1nf, rcl:C-EU025-025X050
- added C_BYP1: 0.1nf, rcl:C-EU025-025X050
- added D1, D2: 1N4148DO35-10, diode:1N4148DO35-10
- added K1: G5LE, relay:G5LE
- added R7: 10k, rcl:R-EU_0207/10
- added RA1: (no value), con-ptr500:AK500/3
- added T2: (no value), transistor:BC548-NPN-TO92-CBE
- added U2: ACS712ELCTR-05B-T, Allegro_By_element14_Batch_1:ACS712ELCTR-05B-T
Connections:
- removed net N$17: IC2.PD3(INT1), R4.1, X1-2.KL
- new net N$28: D2.A, K11.2, T2.C
- new net N$30: R7.1, T2.B
- new net N$31: K12.O, RA1-1.KL
- new net N$32: K12.S, RA1-3.KL
- new net N$33: IC2.PD7(AIN1)
- new net N$34: K12.P, U2.IP-, U2.IP-_2
- new net N$35: RA1-2.KL, U2.IP+, U2.IP+_2
- new net N$36: CF1.1, U2.FILTER
- new net N$37: IC2.PC5(ADC5/SCL), U2.VIOUT
- net GND: now also CF1.2, C_BYP1.2, T2.E, U2.GND; no longer X1-1.KL
- net N$10: now also D1.A
- net N$25: now also IC2.PC4(ADC4/SDA); no longer IC2.PD7(AIN1)
- net VCC: now also C_BYP1.1, D1.C, D2.C, K11.1, U2.VCC; no longer R4.2

Commit message: fix
Parts:
- removed FUENTE: (no value), con-ptr500:AK500/2
- renumbered TERM1 to SERIAL
Connections:
- removed net N$6: IC2.PB4(MISO), ICSP.3, U$1.SI
- new net N$38: IC2.PB4(MISO), ICSP.1, U$1.SI
- net GND: no longer FUENTE-1.KL
- net N$4: now also IC2.PB0(ICP); no longer IC2.PB2(SS/OC1B)
- net N$7: now also ICSP.3; no longer ICSP.2
- net VCC: now also ICSP.2; no longer FUENTE-2.KL, ICSP.1

Commit message: fix
Parts:
- added D3, D4: 1N4148DO35-10, diode:1N4148DO35-10
Connections:
- new net N$6: D4.A, X2-1.KL
- net GND: now also ICSP.6
- net N$29: now also D3.C, D4.C; no longer X2-1.KL
- net VCC: now also D3.A
Other:
- moved on the sheet: X2-1, X2-2
Changed lines of the file:
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@@
 <part name="C_BYP1" library="rcl" deviceset="C-EU" device="025-025X050" value="0.1nf"/>
 <part name="D2" library="diode" deviceset="1N4148" device="DO35-10"/>
+<part name="GND6" library="supply1" deviceset="GND" device=""/>
+<part name="D3" library="diode" deviceset="1N4148" device="DO35-10"/>
+<part name="D4" library="diode" deviceset="1N4148" device="DO35-10"/>
 </parts>
 <sheets>
@@
 <instance part="GND13" gate="1" x="-279.4" y="322.58"/>
 <instance part="P+12" gate="VCC" x="-264.16" y="342.9"/>
-<instance part="X2" gate="-1" x="-304.8" y="337.82"/>
-<instance part="X2" gate="-2" x="-304.8" y="332.74"/>
+<instance part="X2" gate="-1" x="-317.5" y="335.28"/>
+<instance part="X2" gate="-2" x="-317.5" y="330.2"/>
 <instance part="C6" gate="G$1" x="-266.7" y="332.74"/>
 <instance part="C7" gate="G$1" x="-294.64" y="332.74"/>
@@
 <instance part="C_BYP1" gate="G$1" x="-127" y="469.9"/>
 <instance part="D2" gate="G$1" x="-185.42" y="467.36" rot="R90"/>
+<instance part="GND6" gate="1" x="-205.74" y="228.6"/>
+<instance part="D3" gate="G$1" x="-279.4" y="353.06" rot="R180"/>
+<instance part="D4" gate="G$1" x="-304.8" y="337.82"/>
 </instances>
 <busses>
@@
 <pinref part="C6" gate="G$1" pin="1"/>
 <wire x1="-266.7" y1="335.28" x2="-266.7" y2="337.82" width="0.1524" layer="91"/>
+<pinref part="D3" gate="G$1" pin="A"/>
+<wire x1="-276.86" y1="353.06" x2="-266.7" y2="353.06" width="0.1524" layer="91"/>
+<wire x1="-266.7" y1="353.06" x2="-266.7" y2="337.82" width="0.1524" layer="91"/>
 </segment>
 <segment>
@@
 <wire x1="-279.4" y1="327.66" x2="-287.02" y2="327.66" width="0.1524" layer="91"/>
 <wire x1="-287.02" y1="327.66" x2="-287.02" y2="325.12" width="0.1524" layer="91"/>
-<wire x1="-299.72" y1="325.12" x2="-294.64" y2="325.12" width="0.1524" layer="91"/>
-<pinref part="X2" gate="-2" pin="KL"/>
-<wire x1="-299.72" y1="332.74" x2="-299.72" y2="325.12" width="0.1524" layer="91"/>
 <pinref part="C7" gate="G$1" pin="2"/>
 <wire x1="-294.64" y1="327.66" x2="-294.64" y2="325.12" width="0.1524" layer="91"/>
 <wire x1="-287.02" y1="325.12" x2="-294.64" y2="325.12" width="0.1524" layer="91"/>
+<wire x1="-294.64" y1="325.12" x2="-309.88" y2="325.12" width="0.1524" layer="91"/>
+<wire x1="-309.88" y1="325.12" x2="-309.88" y2="330.2" width="0.1524" layer="91"/>
+<pinref part="X2" gate="-2" pin="KL"/>
+<wire x1="-309.88" y1="330.2" x2="-312.42" y2="330.2" width="0.1524" layer="91"/>
 </segment>
 <segment>
@@
 <wire x1="-129.54" y1="462.28" x2="-129.54" y2="444.5" width="0.1524" layer="91"/>
 <wire x1="-129.54" y1="444.5" x2="-124.46" y2="444.5" width="0.1524" layer="91"/>
+</segment>
+<segment>
+<pinref part="ICSP" gate="A" pin="6"/>
+<pinref part="GND6" gate="1" pin="GND"/>
+<wire x1="-215.9" y1="233.68" x2="-205.74" y2="233.68" width="0.1524" layer="91"/>
+<wire x1="-205.74" y1="233.68" x2="-205.74" y2="231.14" width="0.1524" layer="91"/>
 </segment>
 </net>
@@
 <segment>
 <pinref part="IC1" gate="A1" pin="VI"/>
-<pinref part="X2" gate="-1" pin="KL"/>
 <wire x1="-289.56" y1="337.82" x2="-294.64" y2="337.82" width="0.1524" layer="91"/>
 <pinref part="C7" gate="G$1" pin="1"/>
-<wire x1="-294.64" y1="337.82" x2="-299.72" y2="337.82" width="0.1524" layer="91"/>
 <wire x1="-294.64" y1="335.28" x2="-294.64" y2="337.82" width="0.1524" layer="91"/>
+<pinref part="D3" gate="G$1" pin="C"/>
+<wire x1="-281.94" y1="353.06" x2="-294.64" y2="353.06" width="0.1524" layer="91"/>
+<wire x1="-294.64" y1="353.06" x2="-294.64" y2="337.82" width="0.1524" layer="91"/>
+<pinref part="D4" gate="G$1" pin="C"/>
+<wire x1="-302.26" y1="337.82" x2="-294.64" y2="337.82" width="0.1524" layer="91"/>
 </segment>
 </net>
@@
 </segment>
 </net>
+<net name="N$6" class="0">
+<segment>
+<pinref part="X2" gate="-1" pin="KL"/>
+<wire x1="-312.42" y1="335.28" x2="-312.42" y2="337.82" width="0.1524" layer="91"/>
+<pinref part="D4" gate="G$1" pin="A"/>
+<wire x1="-312.42" y1="337.82" x2="-307.34" y2="337.82" width="0.1524" layer="91"/>
+</segment>
+</net>

Commit message: fix
Parts:
- C7: value .1nf -> 100uf
Changed lines of the file:
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@@
 <part name="X2" library="con-ptr500" deviceset="AK500/2" device=""/>
 <part name="C6" library="rcl" deviceset="C-EU" device="025-025X050" value=".1nf"/>
-<part name="C7" library="rcl" deviceset="C-EU" device="025-025X050" value=".1nf"/>
+<part name="C7" library="rcl" deviceset="C-EU" device="025-025X050" value="100uf"/>
 <part name="D1" library="diode" deviceset="1N4148" device="DO35-10"/>
 <part name="K1" library="relay" deviceset="G5LE" device=""/>

Commit message: se creo el archivo board
Parts:
- removed C6: .1nf, rcl:C-EU025-025X050
- removed C7: 100uf, rcl:C-EU025-025X050
- removed X2: (no value), con-ptr500:AK500/2
- added C_VCCIN, C_VCCOUT: .1nf, rcl:C-EU025-025X050
- added LED1: (no value), adafruit:LED3MM
- added R4: 1k, rcl:R-EU_0207/10
- added VCC: (no value), con-ptr500:AK500/2
- renumbered C5 to C_UP, Q1 to Q_UP, Q2 to Q_MCP
Connections:
- new net N$17: LED1.C, R4.2
- net GND: now also C_VCCIN.2, C_VCCOUT.2, R4.1, VCC-2.KL; no longer C6.2, C7.2, X2-2.KL
- net N$29: now also C_VCCIN.1; no longer C7.1
- net N$6: now also VCC-1.KL; no longer X2-1.KL
- net VCC: now also C_VCCOUT.1, LED1.A; no longer C6.1
Other:
- moved on the sheet: D3, D4, IC1

Commit message: fix
Parts:
- removed D4: 1N4148DO35-10, diode:1N4148DO35-10
- added D5: 1N4004, diode:1N4004
- D3: value 1N4148DO35-10 -> 1N4004; device diode:1N4148DO35-10 -> diode:1N4004
- LED1: value (none) -> Fuente
Connections:
- new net N$41: C_VCCIN.1, D3.C, D5.C, IC1.VI
- net GND: now also VCC-1.KL; no longer VCC-2.KL
- net N$25: now also IC2.PB1(OC1A); no longer IC2.PC4(ADC4/SDA)
- net N$29: now also D5.A, VCC-2.KL; no longer C_VCCIN.1, D3.C, D4.C, IC1.VI
- net N$33: now also R7.2
- net N$37: no longer IC2.PC5(ADC5/SCL)
- net N$6: now also IC2.PB2(SS/OC1B); no longer D4.A, VCC-1.KL
Other:
- moved on the sheet: VCC-1, VCC-2
Changed lines of the file:
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@@
 <part name="D2" library="diode" deviceset="1N4148" device="DO35-10"/>
 <part name="GND6" library="supply1" deviceset="GND" device=""/>
-<part name="D3" library="diode" deviceset="1N4148" device="DO35-10"/>
-<part name="D4" library="diode" deviceset="1N4148" device="DO35-10"/>
-<part name="LED1" library="adafruit" deviceset="LED" device="3MM"/>
+<part name="LED1" library="adafruit" deviceset="LED" device="3MM" value="Fuente"/>
 <part name="R4" library="rcl" deviceset="R-EU_" device="0207/10" value="1k"/>
+<part name="D5" library="diode" deviceset="1N4004" device=""/>
+<part name="GND7" library="supply1" deviceset="GND" device=""/>
+<part name="D3" library="diode" deviceset="1N4004" device=""/>
 </parts>
 <sheets>
@@
 <instance part="GND13" gate="1" x="-317.5" y="330.2"/>
 <instance part="P+12" gate="VCC" x="-281.94" y="365.76"/>
-<instance part="VCC" gate="-1" x="-355.6" y="358.14"/>
-<instance part="VCC" gate="-2" x="-355.6" y="353.06"/>
+<instance part="VCC" gate="-1" x="-370.84" y="370.84"/>
+<instance part="VCC" gate="-2" x="-370.84" y="365.76"/>
 <instance part="C_VCCOUT" gate="G$1" x="-304.8" y="355.6"/>
 <instance part="C_VCCIN" gate="G$1" x="-332.74" y="355.6"/>
@@
 <instance part="D2" gate="G$1" x="-185.42" y="467.36" rot="R90"/>
 <instance part="GND6" gate="1" x="-205.74" y="228.6"/>
-<instance part="D3" gate="G$1" x="-317.5" y="375.92" rot="R180"/>
-<instance part="D4" gate="G$1" x="-342.9" y="360.68"/>
 <instance part="LED1" gate="G$1" x="-294.64" y="355.6"/>
 <instance part="R4" gate="G$1" x="-294.64" y="342.9" rot="R90"/>
+<instance part="D5" gate="1" x="-355.6" y="365.76"/>
+<instance part="GND7" gate="1" x="-360.68" y="375.92" rot="R180"/>
+<instance part="D3" gate="1" x="-320.04" y="375.92" rot="R180"/>
 </instances>
 <busses>
@@
 <pinref part="C_VCCOUT" gate="G$1" pin="1"/>
 <wire x1="-304.8" y1="358.14" x2="-304.8" y2="360.68" width="0.1524" layer="91"/>
-<pinref part="D3" gate="G$1" pin="A"/>
-<wire x1="-314.96" y1="375.92" x2="-304.8" y2="375.92" width="0.1524" layer="91"/>
 <wire x1="-304.8" y1="375.92" x2="-304.8" y2="360.68" width="0.1524" layer="91"/>
 <pinref part="LED1" gate="G$1" pin="A"/>
 <wire x1="-294.64" y1="360.68" x2="-294.64" y2="358.14" width="0.1524" layer="91"/>
+<pinref part="D3" gate="1" pin="A"/>
+<wire x1="-317.5" y1="375.92" x2="-304.8" y2="375.92" width="0.1524" layer="91"/>
 </segment>
 <segment>
@@
 <wire x1="-332.74" y1="350.52" x2="-332.74" y2="347.98" width="0.1524" layer="91"/>
 <wire x1="-325.12" y1="347.98" x2="-332.74" y2="347.98" width="0.1524" layer="91"/>
-<wire x1="-332.74" y1="347.98" x2="-347.98" y2="347.98" width="0.1524" layer="91"/>
-<wire x1="-347.98" y1="347.98" x2="-347.98" y2="353.06" width="0.1524" layer="91"/>
-<pinref part="VCC" gate="-2" pin="KL"/>
-<wire x1="-347.98" y1="353.06" x2="-350.52" y2="353.06" width="0.1524" layer="91"/>
 <pinref part="R4" gate="G$1" pin="1"/>
 <wire x1="-294.64" y1="337.82" x2="-317.5" y2="337.82" width="0.1524" layer="91"/>
@@
 <wire x1="-215.9" y1="233.68" x2="-205.74" y2="233.68" width="0.1524" layer="91"/>
 <wire x1="-205.74" y1="233.68" x2="-205.74" y2="231.14" width="0.1524" layer="91"/>
+</segment>
+<segment>
+<pinref part="VCC" gate="-1" pin="KL"/>
+<pinref part="GND7" gate="1" pin="GND"/>
+<wire x1="-365.76" y1="370.84" x2="-360.68" y2="370.84" width="0.1524" layer="91"/>
+<wire x1="-360.68" y1="370.84" x2="-360.68" y2="373.38" width="0.1524" layer="91"/>
 </segment>
 </net>
@@
 <segment>
 <pinref part="IC2" gate="G$1" pin="PD6(AIN0)"/>
+<wire x1="-200.66" y1="284.48" x2="-193.04" y2="284.48" width="0.1524" layer="91"/>
 <pinref part="R5" gate="G$1" pin="2"/>
-<wire x1="-200.66" y1="284.48" x2="-193.04" y2="284.48" width="0.1524" layer="91"/>
-<wire x1="-193.04" y1="284.48" x2="-193.04" y2="360.68" width="0.1524" layer="91"/>
+<wire x1="-193.04" y1="360.68" x2="-193.04" y2="284.48" width="0.1524" layer="91"/>
 </segment>
 </net>
@@
 <wire x1="-68.58" y1="378.46" x2="-68.58" y2="340.36" width="0.1524" layer="91"/>
 <wire x1="-68.58" y1="340.36" x2="-180.34" y2="340.36" width="0.1524" layer="91"/>
-<pinref part="IC2" gate="G$1" pin="PC4(ADC4/SDA)"/>
-<wire x1="-200.66" y1="312.42" x2="-180.34" y2="312.42" width="0.1524" layer="91"/>
-<wire x1="-180.34" y1="312.42" x2="-180.34" y2="340.36" width="0.1524" layer="91"/>
-</segment>
-</net>
-<net name="N$29" class="0">
-<segment>
-<pinref part="IC1" gate="A1" pin="VI"/>
-<wire x1="-327.66" y1="360.68" x2="-332.74" y2="360.68" width="0.1524" layer="91"/>
-<pinref part="C_VCCIN" gate="G$1" pin="1"/>
-<wire x1="-332.74" y1="358.14" x2="-332.74" y2="360.68" width="0.1524" layer="91"/>
-<pinref part="D3" gate="G$1" pin="C"/>
-<wire x1="-320.04" y1="375.92" x2="-332.74" y2="375.92" width="0.1524" layer="91"/>
-<wire x1="-332.74" y1="375.92" x2="-332.74" y2="360.68" width="0.1524" layer="91"/>
-<pinref part="D4" gate="G$1" pin="C"/>
-<wire x1="-340.36" y1="360.68" x2="-332.74" y2="360.68" width="0.1524" layer="91"/>
+<wire x1="-180.34" y1="287.02" x2="-180.34" y2="340.36" width="0.1524" layer="91"/>
+<wire x1="-180.34" y1="287.02" x2="-187.96" y2="287.02" width="0.1524" layer="91"/>
+<wire x1="-187.96" y1="287.02" x2="-187.96" y2="274.32" width="0.1524" layer="91"/>
+<pinref part="IC2" gate="G$1" pin="PB1(OC1A)"/>
+<wire x1="-187.96" y1="274.32" x2="-200.66" y2="274.32" width="0.1524" layer="91"/>
 </segment>
 </net>
@@
 <wire x1="-71.12" y1="434.34" x2="-182.88" y2="434.34" width="0.1524" layer="91"/>
 <wire x1="-182.88" y1="406.4" x2="-182.88" y2="434.34" width="0.1524" layer="91"/>
-<pinref part="IC2" gate="G$1" pin="PC5(ADC5/SCL)"/>
-<wire x1="-195.58" y1="309.88" x2="-200.66" y2="309.88" width="0.1524" layer="91"/>
 <wire x1="-182.88" y1="406.4" x2="-195.58" y2="406.4" width="0.1524" layer="91"/>
-<wire x1="-195.58" y1="406.4" x2="-195.58" y2="309.88" width="0.1524" layer="91"/>
 </segment>
 </net>
 <net name="N$33" class="0">
 <segment>
-<wire x1="-193.04" y1="454.66" x2="-200.66" y2="454.66" width="0.1524" layer="91"/>
 <wire x1="-200.66" y1="454.66" x2="-200.66" y2="396.24" width="0.1524" layer="91"/>
 <wire x1="-200.66" y1="396.24" x2="-165.1" y2="396.24" width="0.1524" layer="91"/>
@@
 <wire x1="-165.1" y1="325.12" x2="-172.72" y2="325.12" width="0.1524" layer="91"/>
 <wire x1="-172.72" y1="325.12" x2="-172.72" y2="284.48" width="0.1524" layer="91"/>
-<wire x1="-172.72" y1="284.48" x2="-190.5" y2="284.48" width="0.1524" layer="91"/>
-<wire x1="-190.5" y1="284.48" x2="-193.04" y2="281.94" width="0.1524" layer="91"/>
+<pinref part="R7" gate="G$1" pin="2"/>
+<wire x1="-200.66" y1="454.66" x2="-195.58" y2="454.66" width="0.1524" layer="91"/>
+<wire x1="-172.72" y1="284.48" x2="-185.42" y2="284.48" width="0.1524" layer="91"/>
+<wire x1="-185.42" y1="284.48" x2="-185.42" y2="281.94" width="0.1524" layer="91"/>
 <pinref part="IC2" gate="G$1" pin="PD7(AIN1)"/>
-<wire x1="-193.04" y1="281.94" x2="-200.66" y2="281.94" width="0.1524" layer="91"/>
+<wire x1="-185.42" y1="281.94" x2="-200.66" y2="281.94" width="0.1524" layer="91"/>
 </segment>
 </net>
@@
 </segment>
 </net>
-<net name="N$6" class="0">
-<segment>
-<pinref part="VCC" gate="-1" pin="KL"/>
-<wire x1="-350.52" y1="358.14" x2="-350.52" y2="360.68" width="0.1524" layer="91"/>
-<pinref part="D4" gate="G$1" pin="A"/>
-<wire x1="-350.52" y1="360.68" x2="-345.44" y2="360.68" width="0.1524" layer="91"/>
-</segment>
-</net>
 <net name="N$17" class="0">
 <segment>
@@
 </segment>
 </net>
+<net name="N$41" class="0">
+<segment>
+<wire x1="-335.28" y1="365.76" x2="-335.28" y2="360.68" width="0.1524" layer="91"/>
+<pinref part="D5" gate="1" pin="C"/>
+<wire x1="-353.06" y1="365.76" x2="-335.28" y2="365.76" width="0.1524" layer="91"/>
+<pinref part="IC1" gate="A1" pin="VI"/>
+<wire x1="-327.66" y1="360.68" x2="-332.74" y2="360.68" width="0.1524" layer="91"/>
+<pinref part="C_VCCIN" gate="G$1" pin="1"/>
+<wire x1="-332.74" y1="360.68" x2="-335.28" y2="360.68" width="0.1524" layer="91"/>
+<wire x1="-332.74" y1="358.14" x2="-332.74" y2="360.68" width="0.1524" layer="91"/>
+<wire x1="-332.74" y1="375.92" x2="-332.74" y2="360.68" width="0.1524" layer="91"/>
+<pinref part="D3" gate="1" pin="C"/>
+<wire x1="-332.74" y1="375.92" x2="-322.58" y2="375.92" width="0.1524" layer="91"/>
+</segment>
+</net>
+<net name="N$29" class="0">
+<segment>
+<pinref part="VCC" gate="-2" pin="KL"/>
+<pinref part="D5" gate="1" pin="A"/>
+<wire x1="-365.76" y1="365.76" x2="-358.14" y2="365.76" width="0.1524" layer="91"/>
+</segment>
+</net>
+<net name="N$6" class="0">
+<segment>
+<pinref part="IC2" gate="G$1" pin="PB2(SS/OC1B)"/>
+<wire x1="-200.66" y1="271.78" x2="-195.58" y2="271.78" width="0.1524" layer="91"/>
+<wire x1="-195.58" y1="271.78" x2="-195.58" y2="375.92" width="0.1524" layer="91"/>
+</segment>
+</net>

Commit message: fix
Parts:
- SERIAL: device pinhead:PINHD-1X2 -> con-ptr500:AK500/2
Connections:
- removed net N$37: U2.VIOUT
- net N$22: now also SERIAL-2.KL; no longer SERIAL.1
- net N$23: now also SERIAL-1.KL; no longer SERIAL.2
- net N$6: now also U2.VIOUT
Changed lines of the file:
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@@
 <part name="GND10" library="supply1" deviceset="GND" device=""/>
 <part name="R6" library="rcl" deviceset="R-EU_" device="0207/10" value="10k"/>
-<part name="SERIAL" library="pinhead" deviceset="PINHD-1X2" device=""/>
 <part name="ICSP" library="pinhead" deviceset="PINHD-2X3" device=""/>
 <part name="P+10" library="supply1" deviceset="VCC" device="" value="+5V"/>
@@
 <part name="GND7" library="supply1" deviceset="GND" device=""/>
 <part name="D3" library="diode" deviceset="1N4004" device=""/>
+<part name="SERIAL" library="con-ptr500" deviceset="AK500/2" device=""/>
 </parts>
 <sheets>
@@
 <instance part="GND10" gate="1" x="-200.66" y="347.98"/>
 <instance part="R6" gate="G$1" x="-251.46" y="332.74" rot="R90"/>
-<instance part="SERIAL" gate="G$1" x="-182.88" y="297.18"/>
 <instance part="ICSP" gate="A" x="-220.98" y="236.22"/>
 <instance part="P+10" gate="VCC" x="-205.74" y="243.84"/>
@@
 <instance part="GND7" gate="1" x="-360.68" y="375.92" rot="R180"/>
 <instance part="D3" gate="1" x="-320.04" y="375.92" rot="R180"/>
+<instance part="SERIAL" gate="-1" x="-185.42" y="294.64" rot="R180"/>
+<instance part="SERIAL" gate="-2" x="-185.42" y="299.72" rot="R180"/>
 </instances>
 <busses>
@@
 </segment>
 </net>
-<net name="N$22" class="0">
-<segment>
-<pinref part="IC2" gate="G$1" pin="PD0(RXD)"/>
-<pinref part="SERIAL" gate="G$1" pin="1"/>
-<wire x1="-200.66" y1="299.72" x2="-185.42" y2="299.72" width="0.1524" layer="91"/>
-</segment>
-</net>
-<net name="N$23" class="0">
-<segment>
-<pinref part="IC2" gate="G$1" pin="PD1(TXD)"/>
-<pinref part="SERIAL" gate="G$1" pin="2"/>
-<wire x1="-200.66" y1="297.18" x2="-185.42" y2="297.18" width="0.1524" layer="91"/>
-</segment>
-</net>
 <net name="N$24" class="0">
 <segment>
@@
 </segment>
 </net>
-<net name="N$37" class="0">
-<segment>
-<pinref part="U2" gate="A" pin="VIOUT"/>
-<wire x1="-73.66" y1="472.44" x2="-71.12" y2="472.44" width="0.1524" layer="91"/>
-<wire x1="-71.12" y1="472.44" x2="-71.12" y2="434.34" width="0.1524" layer="91"/>
-<wire x1="-71.12" y1="434.34" x2="-182.88" y2="434.34" width="0.1524" layer="91"/>
-<wire x1="-182.88" y1="406.4" x2="-182.88" y2="434.34" width="0.1524" layer="91"/>
-<wire x1="-182.88" y1="406.4" x2="-195.58" y2="406.4" width="0.1524" layer="91"/>
-</segment>
-</net>
 <net name="N$33" class="0">
 <segment>
@@
 <pinref part="IC2" gate="G$1" pin="PB2(SS/OC1B)"/>
 <wire x1="-200.66" y1="271.78" x2="-195.58" y2="271.78" width="0.1524" layer="91"/>
-<wire x1="-195.58" y1="271.78" x2="-195.58" y2="375.92" width="0.1524" layer="91"/>
-</segment>
-</net>
+<wire x1="-195.58" y1="271.78" x2="-195.58" y2="406.4" width="0.1524" layer="91"/>
+<pinref part="U2" gate="A" pin="VIOUT"/>
+<wire x1="-73.66" y1="472.44" x2="-71.12" y2="472.44" width="0.1524" layer="91"/>
+<wire x1="-71.12" y1="472.44" x2="-71.12" y2="434.34" width="0.1524" layer="91"/>
+<wire x1="-71.12" y1="434.34" x2="-182.88" y2="434.34" width="0.1524" layer="91"/>
+<wire x1="-182.88" y1="406.4" x2="-182.88" y2="434.34" width="0.1524" layer="91"/>
+<wire x1="-182.88" y1="406.4" x2="-195.58" y2="406.4" width="0.1524" layer="91"/>
+</segment>
+</net>
+<net name="N$22" class="0">
+<segment>
+<pinref part="IC2" gate="G$1" pin="PD0(RXD)"/>
+<pinref part="SERIAL" gate="-2" pin="KL"/>
+<wire x1="-200.66" y1="299.72" x2="-190.5" y2="299.72" width="0.1524" layer="91"/>
+</segment>
+</net>
+<net name="N$23" class="0">
+<segment>
+<pinref part="IC2" gate="G$1" pin="PD1(TXD)"/>
+<pinref part="SERIAL" gate="-1" pin="KL"/>
+<wire x1="-200.66" y1="297.18" x2="-190.5" y2="297.18" width="0.1524" layer="91"/>
+<wire x1="-190.5" y1="297.18" x2="-190.5" y2="294.64" width="0.1524" layer="91"/>
+</segment>
+</net>
