File: can.sch (EAGLE design)
At the start: 46 parts, among them IC1 7805TV, IC2 MEGA8-P, K1 G5LE, K2 G5LE, U1 ACS712ELCTR-05B-T, U2 ACS712ELCTR-05B-T

Commit message: fix
Changed lines of the file:
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@@
-</segment>
-<segment>
-<pinref part="GND9" gate="1" pin="GND"/>
-<pinref part="T1" gate="G$1" pin="E"/>
-<wire x1="-175.26" y1="353.06" x2="-175.26" y2="355.6" width="0.1524" layer="91"/>
 </segment>
 <segment>
@@
 <pinref part="GND11" gate="1" pin="GND"/>
 <wire x1="-106.68" y1="355.6" x2="-109.22" y2="355.6" width="0.1524" layer="91"/>
-</segment>
-<segment>
-<pinref part="CF" gate="G$1" pin="2"/>
-<pinref part="GND12" gate="1" pin="GND"/>
-<wire x1="-121.92" y1="353.06" x2="-121.92" y2="350.52" width="0.1524" layer="91"/>
-<pinref part="C_BYP" gate="G$1" pin="2"/>
-<wire x1="-124.46" y1="370.84" x2="-127" y2="368.3" width="0.1524" layer="91"/>
-<wire x1="-127" y1="368.3" x2="-127" y2="350.52" width="0.1524" layer="91"/>
-<wire x1="-127" y1="350.52" x2="-121.92" y2="350.52" width="0.1524" layer="91"/>
 </segment>
 <segment>
@@
 <wire x1="-360.68" y1="370.84" x2="-360.68" y2="373.38" width="0.1524" layer="91"/>
 </segment>
+<segment>
+<pinref part="GND9" gate="1" pin="GND"/>
+<pinref part="T1" gate="G$1" pin="E"/>
+<wire x1="-175.26" y1="353.06" x2="-175.26" y2="355.6" width="0.1524" layer="91"/>
+</segment>
+<segment>
+<pinref part="CF" gate="G$1" pin="2"/>
+<pinref part="GND12" gate="1" pin="GND"/>
+<wire x1="-121.92" y1="353.06" x2="-121.92" y2="350.52" width="0.1524" layer="91"/>
+<pinref part="C_BYP" gate="G$1" pin="2"/>
+<wire x1="-124.46" y1="370.84" x2="-127" y2="368.3" width="0.1524" layer="91"/>
+<wire x1="-127" y1="368.3" x2="-127" y2="350.52" width="0.1524" layer="91"/>
+<wire x1="-121.92" y1="350.52" x2="-127" y2="350.52" width="0.1524" layer="91"/>
+</segment>
 </net>
