File: can.brd (EAGLE design)
At the start: 160 x 100 mm, 46 parts, among them IC1 7805TV, IC2 MEGA8-P, K1 G5LE, K2 G5LE, U1 ACS712ELCTR-05B-T, U2 ACS712ELCTR-05B-T

Commit message: se creo el archivo board
Parts:
- moved U$1 174.5 mm to (96.5, 38.1), turned to 90 degrees
- moved R2 166.3 mm to (83.8, 27.9), turned to 180 degrees
- moved U$2 165.8 mm to (96.5, 53.3)
- moved R1 165.1 mm to (96.5, 27.9)
- moved CAN 163.9 mm to (113.0, 53.3), turned to 270 degrees
- moved TERM 151.2 mm to (99.1, 61.0), turned to 90 degrees
- moved Q_MCP 147.6 mm to (114.3, 38.1), turned to 270 degrees
- moved C1 137.2 mm to (57.1, 53.3)
- moved C4 137.0 mm to (106.7, 43.2), turned to 180 degrees
- moved C3 134.7 mm to (108.0, 31.8), turned to 180 degrees
- moved ICSP 126.1 mm to (83.8, 48.3), turned to 180 degrees
- moved R3 121.7 mm to (104.1, 57.1), turned to 90 degrees
- moved C_UP 115.7 mm to (55.9, 62.2), turned to 90 degrees
- moved IC2 111.7 mm to (73.7, 74.9)
- moved SERIAL 110.1 mm to (66.0, 91.4)
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
Commit message: fix
Parts:
- removed D4: 1N4148DO35-10, diode:DO35-10
- added D5: 1N4004, diode:DO41-10
- D3: value 1N4148DO35-10 -> 1N4004; device diode:DO35-10 -> diode:DO41-10
- LED1: value (none) -> Fuente
- moved R6 72.0 mm to (101.6, 45.1), turned to 180 degrees
- moved U2 58.7 mm to (25.4, 13.3)
- moved SERIAL 57.5 mm to (106.7, 50.8), turned to 180 degrees
- moved U$2 54.6 mm to (66.7, 7.62), turned to 270 degrees
- moved C_BYP 50.8 mm to (23.5, 22.9), turned to 90 degrees
- moved K1 47.0 mm to (24.1, 10.2), flipped to the bottom, turned to 0 degrees
- moved RA1 47.0 mm to (6.35, 10.2), flipped to the bottom, turned to 270 degrees
- moved Q_MCP 46.5 mm to (76.2, 11.4), turned to 180 degrees
- moved C4 46.4 mm to (79.4, 5.71), turned to 90 degrees
- moved R3 46.2 mm to (97.8, 11.4)
- moved D2 45.7 mm to (39.4, 10.2), turned to 90 degrees
- moved CF1 45.7 mm to (27.3, 22.9), turned to 90 degrees
- moved TERM 44.9 mm to (92.7, 16.5), turned to 0 degrees
- moved C3 43.6 mm to (73.0, 5.71), turned to 90 degrees
- moved CAN 42.5 mm to (106.0, 11.4), flipped to the bottom
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Connections:
- new net N$41: C_VCCIN.1, D3.C, D5.C, IC1.1
- net GND: now also VCC.1; no longer VCC.2
- net N$25: now also IC2.15; no longer IC2.27
- net N$29: now also D5.A, VCC.2; no longer C_VCCIN.1, D3.C, D4.C, IC1.1
- net N$33: now also R7.2
- net N$37: no longer IC2.28
- net N$6: now also IC2.16; no longer D4.A, VCC.1
Routing:
- net VCC: track 0.00 -> 327.2 mm, vias 0 -> 6
- net GND: track 0.00 -> 323.5 mm, vias 0 -> 2
- net B3: track 0.00 -> 85.9 mm, vias 0 -> 2
- net B2: track 0.00 -> 73.1 mm, vias 0 -> 2
- net N$7: track 0.00 -> 69.0 mm
- net N$3: track 0.00 -> 68.1 mm
- net N$25: track 0.00 -> 65.3 mm, vias 0 -> 2
- net N$38: track 0.00 -> 64.2 mm
- net B1: track 0.00 -> 60.2 mm, vias 0 -> 2
- net N$14: track 0.00 -> 51.8 mm
- net N$21: track 0.00 -> 49.9 mm
- net B0: track 0.00 -> 48.2 mm, vias 0 -> 2
- net N$5: track 0.00 -> 46.9 mm
- net N$4: track 0.00 -> 39.0 mm, vias 0 -> 2
- net N$30: track 0.00 -> 32.9 mm
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Other:
- board text added: "2016"

Commit message: fix
Parts:
- SERIAL: device pinhead:1X02 -> con-ptr500:AK500/2
- moved SERIAL 26.5 mm to (111.8, 76.8), flipped to the bottom
- moved C_UP 18.9 mm to (97.2, 51.4), turned to 0 degrees
- moved AN1 14.4 mm to (56.5, 71.1)
- moved AN3 14.4 mm to (43.8, 71.1)
- moved AN0 14.4 mm to (62.9, 71.1)
- moved AN2 14.4 mm to (50.2, 71.1)
- moved R5 1.80 mm to (72.4, 44.5)
Connections:
- removed net N$37: U2.7
- net N$22: now also SERIAL.2; no longer SERIAL.1
- net N$23: now also SERIAL.1; no longer SERIAL.2
- net N$6: now also U2.7
Routing:
- net N$6: track 0.00 -> 100.7 mm, vias 0 -> 2
- net GND: track 323.5 -> 401.1 mm
- net N$18: track 19.7 -> 73.6 mm
- net N$20: track 13.8 -> 66.4 mm
- net N$35: track 19.3 -> 66.4 mm
- net N$19: track 13.8 -> 55.2 mm
- net N$31: track 13.5 -> 50.6 mm
- net N$32: track 13.8 -> 38.4 mm
- net N$23: track 6.35 -> 27.4 mm
- net N$22: track 7.25 -> 26.0 mm
- net N$34: track 8.55 -> 25.7 mm
- net N$27: track 6.38 -> 22.7 mm
- net B0: track 48.2 -> 40.2 mm, vias 2 -> 0
- net N$30: track 32.9 -> 39.7 mm
- net N$37: track 5.42 -> 0.00 mm
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Other:
- board size 160 x 100 mm -> 117.5 x 82.9 mm

Commit message: fix
Parts:
- moved D3 23.1 mm to (12.1, 50.8), turned to 180 degrees
- moved D5 18.4 mm to (12.1, 54.6), turned to 180 degrees
- moved LED1 16.3 mm to (21.0, 52.1), turned to 0 degrees
- moved IC1 15.4 mm to (14.0, 62.2)
- moved C_VCCIN 14.5 mm to (27.3, 64.8)
- moved C_VCCOUT 14.1 mm to (27.3, 59.1)
- moved R4 12.3 mm to (21.6, 60.3)
- moved VCC 11.0 mm to (8.26, 62.2)
Routing:
- net GND: track 401.1 -> 359.7 mm, vias 2 -> 0
- net N$41: track 21.5 -> 61.5 mm
- net N$25: track 68.6 -> 73.8 mm, vias 2 -> 0
- net VCC: track 330.9 -> 335.3 mm
- net N$29: track 8.16 -> 5.41 mm
- net N$17: track 3.59 -> 4.71 mm
Other:
- board size 117.5 x 82.9 mm -> 117.5 x 82.2 mm
